File: pdmrazora.kicad_sch (KiCad schematic)
At the start: 8 parts, among them J1 9-6437287-8, J2 M6_VBAT_GND

Commit message: Re-nest PowerCore EMI split with M6 bobbins and vertical SuperSeal
Replace the J2 2.54 mm power header with dual M6 bolt-through bobbins
(22 mm pitch into the VBAT/GND planes), swap J1 to TE 6437288-6 vertical
SuperSeal (Razor 26-pin net pinout unchanged), and split the floorplan so
mega-mcu144 sits west of the connector and PROFET/M6 east of it.

Refresh M1000 from hellen-one mega-mcu144 0.7 so keepout matches silk,
Value stays Module:mega-mcu144/0.7, rotation 0°, aux origin bottom-left.
Shrink Edge.Cuts 150×130 → 124×106 mm (Razor-class). EN/IS long-haul stay
closed; KiCad 8 headers preserved; stem remains pdmrazora.

Co-authored-by: Quintin <quintinbannink42@users.noreply.github.com>
Parts:
- J1: value 9-6437287-8 -> 6437288-6; footprint pdmrazora:TE_9-6437287-8_SuperSeal26 -> pdmrazora:TE_6437288-6_SuperSeal26_V
- J2: footprint Connector_PinHeader_2.54mm:PinHeader_1x02_P2.54mm_Vertical -> pdmrazora:M6_Bolt_Bobbin_Dual
Other:
- note added: "Power entry: M6+ = VBAT, M6- = GND (bolt-through bobbins) Add TVS, reverse protect, fuse, VBATT sense -> IN_VIGN"
- note removed: "Power entry stub: M6+ = VBAT, M6- = GND Add TVS, reverse protect, fuse, VBATT sense -> IN_VIGN"
Changed lines of the file:
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@@
 			)
 		)
-		(property "Value" "9-6437287-8"
+		(property "Value" "6437288-6"
 			(at 100 130 0)
 			(effects
@@
 			)
 		)
-		(property "Footprint" "pdmrazora:TE_9-6437287-8_SuperSeal26"
+		(property "Footprint" "pdmrazora:TE_6437288-6_SuperSeal26_V"
 			(at 100 110 0)
 			(effects
@@
 			)
 		)
-		(property "Datasheet" "https://www.te.com/en/product-9-6437287-8.html"
+		(property "Datasheet" "https://www.te.com/en/product-6437288-6.html"
 			(at 100 110 0)
 			(effects
@@
 			)
 		)
-		(property "Description" "TE/AMP SuperSeal 1.0 26pos RA Au keying1 (9-6437287-8); Link Connector C"
+		(property "Description" "TE/AMP SuperSeal 1.0 26pos VERTICAL Au keying1 (6437288-6); Link Connector C pinout unchanged"
 			(at 100 110 0)
 			(effects
@@
 			)
 		)
-		(property "Footprint" "Connector_PinHeader_2.54mm:PinHeader_1x02_P2.54mm_Vertical"
+		(property "Footprint" "pdmrazora:M6_Bolt_Bobbin_Dual"
 			(at 35 35 0)
 			(effects
@@
 			)
 		)
-		(property "Description" "M6 main power stubs VBAT+ / GND"
+		(property "Description" "Dual M6 bolt-through bobbin terminals VBAT+ / GND, 22 mm pitch"
 			(at 35 35 0)
 			(effects
@@
 		)
 	)
-	(text "Power entry stub:\nM6+ = VBAT, M6- = GND\nAdd TVS, reverse protect, fuse,\nVBATT sense -> IN_VIGN"
+	(text "Power entry:\nM6+ = VBAT, M6- = GND (bolt-through bobbins)\nAdd TVS, reverse protect, fuse,\nVBATT sense -> IN_VIGN"
 		(at 20 105 0)
 		(effects
